Commit message: chore: 세션 잔여 변경 일괄 커밋 (description/hardware/scenario_ui/box_align/docs)
기존 작업트리에 누적돼 있던 잔여 변경 일괄 정리:
- openarmx_description: body_link0_1350 메시(visual/collision) + URDF/xacro/rviz 갱신
- openarmx_hardware: v10_simple_hardware.cpp
- scenario_ui: diagnostics/launch_manager/pick_and_place/scenario_action_client/joint_data/main_window
- pick_and_place(cyclo/pilz): box_align 노드 + package.xml
- docs: issues_and_fixes / user_instructions
- experiments/joint_gain_tuner.py, scenarios/teach_seq 추가

스크래치 제외: v10_simple_hardware.cpp.bak, 임시 RViz 스크린샷, docs/claude-mistake/2026-06-05.md

Co-Authored-By: Claude Opus 4.8 <noreply@anthropic.com>

File: openarmx_ws/src/openarmx_description/urdf/body/openarmx_body_macro.xacro (robot description, xacro)
@@ -23,11 +23,14 @@
         <xacro:openarmx-body-kinematics config="${kinematics_link}" name="${name}" />
         <geometry>
-          <mesh filename="package://${description_pkg}/meshes/body/${body_type}/visual/${name}.dae" scale="1.0 1.0 1.0" />
+          <mesh filename="package://${description_pkg}/meshes/body/${body_type}/visual/body_link0_1350.stl" scale="0.001 0.001 0.001" />
         </geometry>
+        <material name="body_link0_default">
+          <color rgba="0.30 0.32 0.35 1.0"/>
+        </material>
       </visual>
       <collision name="${prefix}${name}_collision">
         <xacro:openarmx-body-kinematics config="${kinematics_link}" name="${name}" />
         <geometry>
-          <mesh filename="package://openarmx_description/meshes/body/${body_type}/collision/${name}_symp.stl" scale="1.0 1.0 1.0" />
+          <mesh filename="package://openarmx_description/meshes/body/${body_type}/collision/body_link0_1350.stl" scale="0.001 0.001 0.001" />
           <!-- <mesh filename="package://openarmx_description/meshes/arm/${arm_type}/collision/${name}.stl" scale="0.001 0.001 0.001" /> -->
         </geometry>

File: openarmx_ws/src/openarmx_description/urdf/robot/openarmx_robot.xacro (robot description, xacro)
@@ -164,5 +164,5 @@
         <xacro:property name="special_connection" value="$(arg special_connection)" />
         <!-- <xacro:property name="connection" value="${special_connection if special_connection != '' else arm_type + '_link7'}" /> -->
-        <xacro:property name="connection" value="${special_connection if special_connection != '' else 'openarm' + '_link7'}" />
+        <xacro:property name="connection" value="${special_connection if special_connection != '' else 'openarmx_link7'}" />
         <xacro:if value="$(eval hand and ee_type == 'openarmx_hand')">
         <xacro:openarmx_hand

File: openarmx_ws/src/openarmx_description/urdf/robot/v10.urdf.xacro (robot description, xacro)
@@ -26,7 +26,7 @@
   <xacro:arg name="left_arm_base_xyz" default="0.0 0.031 0.698" />
   <xacro:arg name="left_arm_base_rpy" default="-1.5708 0 0" /> -->
-  <xacro:arg name="right_arm_base_xyz" default="0.0 -0.031 0.735" />
+  <xacro:arg name="right_arm_base_xyz" default="0.0 -0.031 1.275" />
   <xacro:arg name="right_arm_base_rpy" default="1.5708 0 0" />
-  <xacro:arg name="left_arm_base_xyz" default="0.0 0.031 0.735" />
+  <xacro:arg name="left_arm_base_xyz" default="0.0 0.031 1.275" />
   <xacro:arg name="left_arm_base_rpy" default="-1.5708 0 0" />
   <xacro:arg name="can_fd" default="false" />
@@ -71,9 +71,11 @@
   <!-- Parent frame openarmx_body_link0 only exists in bimanual, so  -->
   <!-- this block is guarded; single-arm v10 stays unchanged.        -->
-  <!-- Extrinsic (2026-06-01 ChArUco recalib, 60deg mount,           -->
-  <!-- board @ base_link (0.35, 0, 0.12) m, roll 180):               -->
+  <!-- Extrinsic (2026-06-05 ChArUco recalib, raised-arm config:     -->
+  <!--   arm_base z=1.275 (+0.54 m vs old), 60deg mount,             -->
+  <!--   board @ openarmx_body_link0 (0.19, 0.175, 0.72) m, roll 180; -->
+  <!--   fresh ChArUco 30-frame PnP solve on kkw cam)               -->
   <!--   body_link0 -> d435_center_link                              -->
-  <!--   t=(0.065430, 0.000987, 0.641921) m                          -->
-  <!--   rpy=(0.6846, 59.7350, 0.4038) deg                           -->
+  <!--   t=(0.062816, 0.020383, 1.183573) m                         -->
+  <!--   rpy=(-0.4588, 59.7955, -0.6353) deg                         -->
   <!-- Mesh visual origin copied from realsense2_description.        -->
   <!-- No collision geometry: planning/control unaffected.           -->
@@ -83,6 +85,6 @@
       <parent link="openarmx_body_link0"/>
       <child link="d435_center_link"/>
-      <origin xyz="0.065430 0.000987 0.641921"
-              rpy="${radians(0.6846)} ${radians(59.7350)} ${radians(0.4038)}"/>
+      <origin xyz="0.062816 0.020383 1.183573"
+              rpy="${radians(-0.4588)} ${radians(59.7955)} ${radians(-0.6353)}"/>
     </joint>
     <link name="d435_center_link">
