Commit message: feat(calibration): D435 카메라를 로봇 모델에 베이크 + RViz 시각화
- v10.urdf.xacro: bimanual 가드 안에 d435_center_link + d435.dae 메쉬 추가
  (캘리브 extrinsic body_link0→d435_center_link, visual only, collision 없음)
- calibration_camera.rviz: 로봇+카메라 모델 + TF 좌표축 전용 RViz 설정
- calibration_bringup_with_camera_tf.launch.py: 중복 static TF/별도 RSP 제거,
  bimanual:=true 기본값 + 전용 rviz 지정
- README.md: 캘리브 절차/결과/시각화/빌드 노트 문서화

Co-Authored-By: Claude Opus 4.8 <noreply@anthropic.com>

File: openarmx_ws/src/openarmx_description/urdf/robot/v10.urdf.xacro (robot description, xacro)
@@ -67,3 +67,30 @@
   control_mode="$(arg control_mode)"
   />
+  <!-- ============================================================= -->
+  <!-- Calibrated D435 center camera (visual-only).                  -->
+  <!-- Parent frame openarmx_body_link0 only exists in bimanual, so  -->
+  <!-- this block is guarded; single-arm v10 stays unchanged.        -->
+  <!-- Extrinsic (2026-05-27 ChArUco calibration, board @ +0.59m):   -->
+  <!--   body_link0 -> d435_center_link                              -->
+  <!--   t=(0.034018, 0.036608, 0.644715) m                          -->
+  <!--   rpy=(-1.4041, 31.0059, -2.1785) deg                         -->
+  <!-- Mesh visual origin copied from realsense2_description.        -->
+  <!-- No collision geometry: planning/control unaffected.           -->
+  <!-- ============================================================= -->
+  <xacro:if value="$(arg bimanual)">
+    <joint name="d435_center_calib_joint" type="fixed">
+      <parent link="openarmx_body_link0"/>
+      <child link="d435_center_link"/>
+      <origin xyz="0.034018 0.036608 0.644715"
+              rpy="${radians(-1.4041)} ${radians(31.0059)} ${radians(-2.1785)}"/>
+    </joint>
+    <link name="d435_center_link">
+      <visual>
+        <origin xyz="0.0043 -0.0175 0" rpy="${pi/2} 0 ${pi/2}"/>
+        <geometry>
+          <mesh filename="package://realsense2_description/meshes/d435.dae"/>
+        </geometry>
+      </visual>
+    </link>
+  </xacro:if>
 </robot>

Commit message: feat(calibration): D435 카메라 마운트 각도 변경 재캘리브 (45°→60°)
마운트 틸트를 60°로 변경 후 ChArUco extrinsic 재캘리브레이션.
틸트 변경은 pitch뿐 아니라 translation(광학중심)도 이동시키므로
숫자 패치가 아닌 6-DOF 재측정 필수. body_link0→d435_center_link
extrinsic을 보유 6개 파일에 동기화.

- v10.urdf.xacro: d435_center_calib_joint origin (pitch 59.735°, z 0.642m)
- calibration/README.md: §1 결과 + 각도 이력(30→45→60)
- calibration_bringup_with_camera_tf.launch.py: docstring 주석
- calibration_camera.rviz: PointCloud2 디스플레이 추가 (정합 확인용)
- yolov8_d435.launch.py: _CAM_TF 갱신 (박스검출 standalone TF)

검증: link-frame pitch≈마운트각(59.735°), 위치 std<0.1mm,
라이브 charuco_board TF가 보드 실측 pose 재현(|Δ|=2.1mm).

문서: docs/issues_and_fixes/2026-06-01_d435_camera_angle_recalibration.md

Co-Authored-By: Claude Opus 4.8 (1M context) <noreply@anthropic.com>

File: openarmx_ws/src/openarmx_description/urdf/robot/v10.urdf.xacro (robot description, xacro)
@@ -71,8 +71,9 @@
   <!-- Parent frame openarmx_body_link0 only exists in bimanual, so  -->
   <!-- this block is guarded; single-arm v10 stays unchanged.        -->
-  <!-- Extrinsic (2026-05-27 ChArUco calibration, board @ +0.59m):   -->
+  <!-- Extrinsic (2026-06-01 ChArUco recalib, 60deg mount,           -->
+  <!-- board @ base_link (0.35, 0, 0.12) m, roll 180):               -->
   <!--   body_link0 -> d435_center_link                              -->
-  <!--   t=(0.034018, 0.036608, 0.644715) m                          -->
-  <!--   rpy=(-1.4041, 31.0059, -2.1785) deg                         -->
+  <!--   t=(0.065430, 0.000987, 0.641921) m                          -->
+  <!--   rpy=(0.6846, 59.7350, 0.4038) deg                           -->
   <!-- Mesh visual origin copied from realsense2_description.        -->
   <!-- No collision geometry: planning/control unaffected.           -->
@@ -82,6 +83,6 @@
       <parent link="openarmx_body_link0"/>
       <child link="d435_center_link"/>
-      <origin xyz="0.034018 0.036608 0.644715"
-              rpy="${radians(-1.4041)} ${radians(31.0059)} ${radians(-2.1785)}"/>
+      <origin xyz="0.065430 0.000987 0.641921"
+              rpy="${radians(0.6846)} ${radians(59.7350)} ${radians(0.4038)}"/>
     </joint>
     <link name="d435_center_link">

Commit message: fix(model): arm-base 31mm를 xacro SSOT로 일원화 + ptp 백엔드 full URDF 런타임 축소
- v10.urdf.xacro arm_base z 1.275→1.244: FK가 실제보다 상수 +31mm 높던
  arm-base 캘리브 오차를 SSOT 한 곳에서 수정(full URDF/TF/IK/전 백엔드 정합).
  좌팔 (0.10,0.10,0.72) 액션 이동 후 엔코더 FK=실측 일치로 라이브 검증완료.
- ptp 새 백엔드(openarmx_ptp_box_align[+_msgs]): /robot_description 구독→
  buildModelFromXML(full)→팔별 buildReducedModel로 7-DOF 단일팔 모델 런타임 생성,
  솔버 URDF 파일 의존(모델 이중화) 제거. Pinocchio DLS IK→단일 JTC 끝점.
- solver URDF(cyclo 전용)도 1.244로 정합.
- 기록: issues_and_fixes 2026-06-07 05:02, claude-mistake 2026-06-06.

Co-Authored-By: Claude Opus 4.8 <noreply@anthropic.com>

File: openarmx_ws/src/openarmx_description/urdf/robot/v10.urdf.xacro (robot description, xacro)
@@ -26,7 +26,10 @@
   <xacro:arg name="left_arm_base_xyz" default="0.0 0.031 0.698" />
   <xacro:arg name="left_arm_base_rpy" default="-1.5708 0 0" /> -->
-  <xacro:arg name="right_arm_base_xyz" default="0.0 -0.031 1.275" />
+  <!-- arm_base z: 1.275 -> 1.244 (-31mm). FK(model) was a constant +31mm above the
+       real arm (5-pt measure ±1mm, pose-independent → arm-base calibration error, not
+       gravity sag). Fixing here (SSOT) makes full URDF/TF/IK/all backends match reality. -->
+  <xacro:arg name="right_arm_base_xyz" default="0.0 -0.031 1.244" />
   <xacro:arg name="right_arm_base_rpy" default="1.5708 0 0" />
-  <xacro:arg name="left_arm_base_xyz" default="0.0 0.031 1.275" />
+  <xacro:arg name="left_arm_base_xyz" default="0.0 0.031 1.244" />
   <xacro:arg name="left_arm_base_rpy" default="-1.5708 0 0" />
   <xacro:arg name="can_fd" default="false" />

File: openarmx_ws/src/pick_and_place/cyclo/openarmx_pick/urdf/openarmx_left_solver.urdf (robot description, URDF)
Before this commit: robot openarmx, 30 links, 29 joints
Links:
- added link d435_center_link; visual mesh filename=package://realsense2_description/meshes/d435.dae
- link openarmx_body_link0: geometry visual mesh filename=package://openarmx_description/meshes/body/v10/visual/body_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 scale=0.001 0.001 0.001
Joints:
- added joint d435_center_calib_joint: type fixed, parent openarmx_body_link0, child d435_center_link, origin xyz=0.062816 0.020383 1.183573 rpy=-0.008007570608149984 1.0436283528762693 -0.011088076737919976
- joint openarmx_left_joint1: limit lower=-3.344396 upper=0.9056039999999999 effort=120 velocity=10.47 -> lower=-3.3161256000000003 upper=1.3962633999999998 effort=120 velocity=10.47
- joint openarmx_left_joint2: limit lower=-3.2707963267948967 upper=0.1292036732051034 effort=120 velocity=10.47 -> lower=-3.1415926267948966 upper=-2.6794896523796297e-08 effort=120 velocity=10.47
- joint openarmx_left_joint3: limit lower=-1.57 upper=1.57 effort=60 velocity=10.47 -> lower=-1.5707963 upper=1.7453293 effort=60 velocity=10.47
- joint openarmx_left_joint4: limit lower=0.0 upper=1.8 effort=60 velocity=10.47 -> lower=0.0 upper=1.9198622 effort=60 velocity=10.47
- joint openarmx_left_joint5: limit lower=-1.5 upper=1.5 effort=14 velocity=10.47 -> lower=-1.5707963 upper=1.5707963 effort=14 velocity=10.47
- joint openarmx_left_joint6: limit lower=-0.75 upper=0.75 effort=14 velocity=10.47 -> lower=-0.6981317 upper=0.6981317 effort=14 velocity=10.47
- joint openarmx_left_joint7: limit lower=-1.4 upper=1.4 effort=14 velocity=10.47 -> lower=-1.3962634 upper=1.3962634 effort=14 velocity=10.47
- joint openarmx_left_openarmx_body_link0_joint: origin xyz=0.0 0.031 0.735 rpy=-1.5708 0 0 -> xyz=0.0 0.031 1.244 rpy=-1.5708 0 0
- joint openarmx_right_openarmx_body_link0_joint: origin xyz=0.0 -0.031 0.735 rpy=1.5708 0 0 -> xyz=0.0 -0.031 1.244 rpy=1.5708 0 0

File: openarmx_ws/src/pick_and_place/cyclo/openarmx_pick/urdf/openarmx_right_solver.urdf (robot description, URDF)
Before this commit: robot openarmx, 30 links, 29 joints
Links:
- added link d435_center_link; visual mesh filename=package://realsense2_description/meshes/d435.dae
- link openarmx_body_link0: geometry visual mesh filename=package://openarmx_description/meshes/body/v10/visual/body_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 scale=0.001 0.001 0.001
Joints:
- added joint d435_center_calib_joint: type fixed, parent openarmx_body_link0, child d435_center_link, origin xyz=0.062816 0.020383 1.183573 rpy=-0.008007570608149984 1.0436283528762693 -0.011088076737919976
- joint openarmx_left_openarmx_body_link0_joint: origin xyz=0.0 0.031 0.735 rpy=-1.5708 0 0 -> xyz=0.0 0.031 1.244 rpy=-1.5708 0 0
- joint openarmx_right_joint1: limit lower=-1.25 upper=3.0 effort=120 velocity=10.47 -> lower=-1.3962634 upper=3.3161256 effort=120 velocity=10.47
- joint openarmx_right_joint2: limit lower=-0.1292036732051034 upper=3.2707963267948967 effort=120 velocity=10.47 -> lower=2.6794896523796297e-08 upper=3.1415926267948966 effort=120 velocity=10.47
- joint openarmx_right_joint3: limit lower=-1.57 upper=1.57 effort=60 velocity=10.47 -> lower=-1.5707963 upper=1.7453293 effort=60 velocity=10.47
- joint openarmx_right_joint4: limit lower=0.0 upper=1.8 effort=60 velocity=10.47 -> lower=0.0 upper=1.9198622 effort=60 velocity=10.47
- joint openarmx_right_joint5: limit lower=-1.5 upper=1.5 effort=14 velocity=10.47 -> lower=-1.5707963 upper=1.5707963 effort=14 velocity=10.47
- joint openarmx_right_joint6: limit lower=-0.75 upper=0.75 effort=14 velocity=10.47 -> lower=-0.6981317 upper=0.6981317 effort=14 velocity=10.47
- joint openarmx_right_joint7: limit lower=-1.4 upper=1.4 effort=14 velocity=10.47 -> lower=-1.3962634 upper=1.3962634 effort=14 velocity=10.47
- joint openarmx_right_openarmx_body_link0_joint: origin xyz=0.0 -0.031 0.735 rpy=1.5708 0 0 -> xyz=0.0 -0.031 1.244 rpy=1.5708 0 0
